Commit message: final

File: assets/model_door2/urdf/model_door2.urdf (robot description, URDF)
Before this commit: robot model_door2, 2 links, 1 joints
Links:
- link link1: mass 0.03 -> 0.01; geometry collision mesh filename=package://model_door2/meshes/link1.STL; visual mesh filename=package://model_door2/meshes/link1.STL
